File: PCB/gpio_2pin_cluster.kicad_sch (KiCad schematic)
At the start: 3 parts, among them Y1 40MHz

Commit message: yeah just read the journal son
Parts:
- removed C11, C12: MATCH, Capacitor_SMD:C_0603_1608Metric, symbol Device:C
- removed Y1: 40MHz, symbol Device:Crystal_GND24
- added C43: 100n, symbol Device:C
- added C44: 10u, symbol Device:C
- added J16: GPIO, symbol Connector_Generic:Conn_01x02
- added J17: REF, Connector_PinHeader_1.00mm:PinHeader_1x02_P1.00mm_Vertical, symbol Connector_Generic:Conn_01x02
Connections:
- net GND: now also C43.1, C44.1, J17.2 (Pin_2)
- new net cGPIO1: J16.1 (Pin_1)
- new net cGPIO2: J16.2 (Pin_2)
- new net cVDD: C43.2, C44.2, J17.1 (Pin_1)
