File: PCB/mcu.kicad_sch (KiCad schematic)
At the start: 1 part, among them U1 ESP32-S3

Commit message: yeah just read the journal son
Changed lines of the file:
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@@
 	)
 	(hierarchical_label "MTCK"
-		(shape bidirectional)
+		(shape input)
 		(at 222.25 134.62 0)
 		(effects
@@
 	)
 	(hierarchical_label "U0RXD"
-		(shape bidirectional)
+		(shape input)
 		(at 222.25 147.32 0)
 		(effects
@@
 	)
 	(hierarchical_label "MTDO"
-		(shape bidirectional)
+		(shape output)
 		(at 222.25 137.16 0)
 		(effects
@@
 	)
 	(hierarchical_label "MTMS"
-		(shape bidirectional)
+		(shape input)
 		(at 222.25 142.24 0)
 		(effects
@@
 	)
 	(hierarchical_label "U0TXD"
-		(shape bidirectional)
+		(shape output)
 		(at 222.25 144.78 0)
 		(effects
@@
 	)
 	(hierarchical_label "MTDI"
-		(shape bidirectional)
+		(shape input)
 		(at 222.25 139.7 0)
 		(effects
@@
 		(dnp no)
 		(fields_autoplaced yes)
-		(property "Reference" "#PWR03"
+		(property "Reference" "#PWR01"
 			(at 190.5 172.72 0)
 			(hide yes)
@@
 			(project "CTR-1"
 				(path "/59fb818d-89a2-4fec-918a-42976325079d/f0c5dac2-e2d5-4bb6-90d4-372b49657e0b"
-					(reference "#PWR03")
+					(reference "#PWR01")
 					(unit 1)
 				)
