File: PCB/CTR-1.kicad_sch (KiCad schematic)
At the start: 44 parts, among them J1 Conn_Coaxial, J2 JTAG, J3 UART, SW1 RST, SW2 BOOT, U1 ESP32-S3, U2 W25Q128JVP, U3 ESP-PSRAM64H, Y1 32kHz, Y2 40MHz

Commit message: schematic polish
Other:
- note added: "(GPIO15)"
- note added: "(GPIO16)"
- note added: "CLK"
- note added: "HPST"
- note added: "JTAG"
- note added: "RTC"
- note added: "UART"
- note added: "USB"
- note added: "{"
- note removed: "10mA {"
- note removed: "40mA {"
- note removed: "CLK {"
- note removed: "RTC {"
- moved on the sheet: C, U1

Commit message: lot of things happened
Parts:
- removed C10, C13, C15, C20, C21, C24, C8, C9: 100n, symbol Device:C
- removed C11, C14, C19: 1u, symbol Device:C
- removed C12: 10u, symbol Device:C
- removed C16, C17, C22, C23, C5, C6: MATCH, symbol Device:C
- removed C18: 10n, symbol Device:C
- removed C7: 22u, symbol Device:C
- removed J1: Conn_Coaxial, symbol Connector:Conn_Coaxial
- removed J2: JTAG, symbol Connector_Generic:Conn_01x04
- removed J3: UART, symbol Connector_Generic:Conn_01x04
- removed L1: MATCH, symbol Device:L
- removed L2: 2n, symbol Device:L
- removed R5, R6, R7, R8: 10k, symbol Device:R
- removed SW1: RST, symbol Switch:SW_Push
- removed SW2: BOOT, symbol Switch:SW_Push
- removed U1: ESP32-S3, Package_DFN_QFN:QFN-56-1EP_7x7mm_P0.4mm_EP4x4mm, symbol MCU_Espressif:ESP32-S3
- removed U2: W25Q128JVP, Package_SON:WSON-8-1EP_6x5mm_P1.27mm_EP3.4x4.3mm, symbol Memory_Flash:W25Q128JVP
- removed U3: ESP-PSRAM64H, Package_SO:SOIC-8_3.9x4.9mm_P1.27mm, symbol Memory_RAM:ESP-PSRAM32
- removed Y1: 32kHz, symbol Device:Crystal_GND24
- removed Y2: 40MHz, symbol Device:Crystal_GND24
- added J1: JTAG, symbol Connector_Generic:Conn_01x04
- added J2: UART, symbol Connector_Generic:Conn_02x02_Counter_Clockwise
- added J3: REF, symbol Connector_Generic:Conn_01x02
- renumbered C to C1, C to C2, C to C3, C to C4, C to C5, C to C6, C to C7, C to C8
Connections:
- net GND: now also J2.3 (Pin_3), J3.2 (Pin_2)
- new net ESP32-S3 MCU/MTCK: J1.1 (Pin_1)
- new net ESP32-S3 MCU/MTDI: J1.3 (Pin_3)
- new net ESP32-S3 MCU/MTDO: J1.2 (Pin_2)
- new net ESP32-S3 MCU/MTMS: J1.4 (Pin_4)
- new net ESP32-S3 MCU/U0RXD: J2.1 (Pin_1)
- new net ESP32-S3 MCU/U0TXD: J2.2 (Pin_2)
- no-connect marks 0 -> 3
Other:
- added sheet ANTENNA (antenna.kicad_sch)
- added sheet DECOUPLING (decoupling.kicad_sch)
- added sheet EN (en_button.kicad_sch)
- added sheet ESP32-S3 MCU (mcu.kicad_sch)
- added sheet GPIO (gpio.kicad_sch)
- added sheet MEMORY (memory.kicad_sch)
- added sheet POWER (power.kicad_sch)
- added sheet STRAPPING (strapping_pins.kicad_sch)
- added sheet USB_C_RECEPTACLE (usb_c_receptacle.kicad_sch)
- added sheet XTAL_32K_RTC (xtal_32k_rtc.kicad_sch)
- added sheet XTAL_40MHZ (xtal_40mhz.kicad_sch)
- note added: "CPU/Digital power for eFuse"
- note added: "FLASH/PSRAM VDD, 3.3V"
- note added: "Internal analog power, for RF/PLL"
- note added: "MAIN +3V3 POWER LINE"
- note added: "RTC Power, stays on in deep sleep"
- note removed: "(GPIO15)"
- note removed: "(GPIO16)"
- note removed: "3V3 if GPIO45 = 1, else 1V8"
- note removed: "BUTTON"
- note removed: "BUTTONS"
- note removed: "CLK"
- note removed: "CRYSTALS"
- note removed: "DECOUPLING"
- note removed: "FLASH/PSRAM"
- note removed: "HPST"
- note removed: "JTAG"
- note removed: "JTAG/UART"
- note removed: "RTC"
- note removed: "UART"
- note removed: "USB"
- note removed: "u.FL ANTENNA CONNECTOR"
- note removed: "{"
- note removed: "}"

Commit message: yeah just read the journal son
Parts:
- removed J1: JTAG, symbol Connector_Generic:Conn_01x04
- removed J2: UART, symbol Connector_Generic:Conn_02x02_Counter_Clockwise
- removed J3: REF, symbol Connector_Generic:Conn_01x02
Connections:
- no-connect marks 3 -> 4
Other:
- sheet USB_C_RECEPTACLE renamed USB_C
- removed sheet POWER
- added sheet JTAG_PINS (jtag_pins.kicad_sch)
- added sheet POWER_MANAGEMENT (power_mgmt.kicad_sch)
- added sheet UART_PINS (uart_pins.kicad_sch)
- sheet GPIO ports: added GPIO33, GPIO34, GPIO35, GPIO36, GPIO37, GPIO38; removed VDD_GPIO
- sheet MEMORY ports: added ~{CE1}, ~{CS0}; removed ~{CE}
- sheet USB_C: file usb_c_receptacle.kicad_sch -> usb_c.kicad_sch

Commit message: big things are happening
Parts:
- removed C1, C2, C3, C4: V, symbol Device:C
- removed C5, C6, C7, C8: V, symbol Device:R
