File: PCB/antenna.kicad_sch (KiCad schematic)
At the start: 4 parts, among them J4 u.FL

Commit message: yeah just read the journal son
Parts:
- renumbered J4 to J1
Changed lines of the file:
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@@
 		(in_pos_files yes)
 		(dnp no)
-		(property "Reference" "J4"
+		(property "Reference" "J1"
 			(at 204.47 120.65 0)
 			(show_name no)
@@
 			(project "CTR-1"
 				(path "/59fb818d-89a2-4fec-918a-42976325079d/4159d440-b4ab-4425-b126-33ca88c5579d"
-					(reference "J4")
+					(reference "J1")
 					(unit 1)
 				)
@@
 		(dnp no)
 		(fields_autoplaced yes)
-		(property "Reference" "#PWR04"
+		(property "Reference" "#PWR02"
 			(at 185.42 143.51 0)
 			(hide yes)
@@
 			(project "CTR-1"
 				(path "/59fb818d-89a2-4fec-918a-42976325079d/4159d440-b4ab-4425-b126-33ca88c5579d"
-					(reference "#PWR04")
+					(reference "#PWR02")
 					(unit 1)
 				)
@@
 		(dnp no)
 		(fields_autoplaced yes)
-		(property "Reference" "#PWR06"
+		(property "Reference" "#PWR04"
 			(at 204.47 143.51 0)
 			(hide yes)
@@
 			(project "CTR-1"
 				(path "/59fb818d-89a2-4fec-918a-42976325079d/4159d440-b4ab-4425-b126-33ca88c5579d"
-					(reference "#PWR06")
+					(reference "#PWR04")
 					(unit 1)
 				)
@@
 		(dnp no)
 		(fields_autoplaced yes)
-		(property "Reference" "#PWR05"
+		(property "Reference" "#PWR03"
 			(at 195.58 143.51 0)
 			(hide yes)
@@
 			(project "CTR-1"
 				(path "/59fb818d-89a2-4fec-918a-42976325079d/4159d440-b4ab-4425-b126-33ca88c5579d"
-					(reference "#PWR05")
-					(unit 1)
-				)
+					(reference "#PWR03")
+					(unit 1)
+				)

Commit message: big things are happening
Parts:
- C10, C9: value MATCH -> 1.8p
- L1: value MATCH -> 2.7n; footprint (none) -> Inductor_SMD:L_0402_1005Metric
Changed lines of the file:
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@@
 			)
 		)
-		(property "Value" "MATCH"
+		(property "Value" "2.7n"
 			(at 193.04 125.73 90)
 			(show_name no)
@@
 				(font
 					(size 1.27 1.27)
-					(color 128 0 0 1)
 				)
 				(justify right)
 			)
 		)
-		(property "Footprint" ""
+		(property "Footprint" "Inductor_SMD:L_0402_1005Metric"
 			(at 190.5 127 0)
 			(hide yes)
@@
 				(path "/59fb818d-89a2-4fec-918a-42976325079d/4159d440-b4ab-4425-b126-33ca88c5579d"
 					(reference "L1")
+					(unit 1)
+				)
+			)
+		)
+	)
+	(symbol
+		(lib_id "Device:C")
+		(at 195.58 132.08 0)
+		(unit 1)
+		(body_style 1)
+		(exclude_from_sim no)
+		(in_bom yes)
+		(on_board yes)
+		(in_pos_files yes)
+		(dnp no)
+		(property "Reference" "C10"
+			(at 195.834 130.81 0)
+			(show_name no)
+			(do_not_autoplace no)
+			(effects
+				(font
+					(size 1.27 1.27)
+				)
+				(justify left bottom)
+			)
+		)
+		(property "Value" "1.8p"
+			(at 195.834 133.35 0)
+			(show_name no)
+			(do_not_autoplace no)
+			(effects
+				(font
+					(size 1.27 1.27)
+				)
+				(justify left top)
+			)
+		)
+		(property "Footprint" "Capacitor_SMD:C_0603_1608Metric"
+			(at 196.5452 135.89 0)
+			(hide yes)
+			(show_name no)
+			(do_not_autoplace no)
+			(effects
+				(font
+					(size 1.27 1.27)
+				)
+			)
+		)
+		(property "Datasheet" ""
+			(at 195.58 132.08 0)
+			(hide yes)
+			(show_name no)
+			(do_not_autoplace no)
+			(effects
+				(font
+					(size 1.27 1.27)
+				)
+			)
+		)
+		(property "Description" "Unpolarized capacitor"
+			(at 195.58 132.08 0)
+			(hide yes)
+			(show_name no)
+			(do_not_autoplace no)
+			(effects
+				(font
+					(size 1.27 1.27)
+				)
+			)
+		)
+		(pin "1"
+		)
+		(pin "2"
+		)
+		(instances
+			(project "CTR-1"
+				(path "/59fb818d-89a2-4fec-918a-42976325079d/4159d440-b4ab-4425-b126-33ca88c5579d"
+					(reference "C10")
 					(unit 1)
 				)
@@
 			)
 		)
-		(property "Value" "MATCH"
+		(property "Value" "1.8p"
 			(at 185.674 133.35 0)
 			(show_name no)
@@
 				(font
 					(size 1.27 1.27)
-					(color 128 0 0 1)
 				)
 				(justify left top)
@@
 					(unit 1)
 				)
-			)
-		)
-	)
-	(symbol
-		(lib_id "Device:C")
-		(at 195.58 132.08 0)
-		(unit 1)
-		(body_style 1)
-		(exclude_from_sim no)
-		(in_bom yes)
-		(on_board yes)
-		(in_pos_files yes)
-		(dnp no)
-		(property "Reference" "C10"
-			(at 195.834 130.81 0)
-			(show_name no)
-			(do_not_autoplace no)
-			(effects
-				(font
-					(size 1.27 1.27)
-				)
-				(justify left bottom)
-			)
-		)
-		(property "Value" "MATCH"
-			(at 195.834 133.35 0)
-			(show_name no)
-			(do_not_autoplace no)
-			(effects
-				(font
-					(size 1.27 1.27)
-					(color 128 0 0 1)
-				)
-				(justify left top)
-			)
-		)
-		(property "Footprint" "Capacitor_SMD:C_0603_1608Metric"
-			(at 196.5452 135.89 0)
-			(hide yes)
-			(show_name no)
-			(do_not_autoplace no)
-			(effects
-				(font
-					(size 1.27 1.27)
-				)
-			)
-		)
-		(property "Datasheet" ""
-			(at 195.58 132.08 0)
-			(hide yes)
-			(show_name no)
-			(do_not_autoplace no)
-			(effects
-				(font
-					(size 1.27 1.27)
-				)
-			)
-		)
-		(property "Description" "Unpolarized capacitor"
-			(at 195.58 132.08 0)
-			(hide yes)
-			(show_name no)
-			(do_not_autoplace no)
-			(effects
-				(font
-					(size 1.27 1.27)
-				)
-			)
-		)
-		(pin "1"
-		)
-		(pin "2"
-		)
-		(instances
-			(project "CTR-1"
-				(path "/59fb818d-89a2-4fec-918a-42976325079d/4159d440-b4ab-4425-b126-33ca88c5579d"
-					(reference "C10")
-					(unit 1)
-				)
