File: PCB/decoupling.kicad_sch (KiCad schematic)
At the start: 9 parts

Commit message: yeah just read the journal son
Parts:
- C36: renamed from C26; footprint Capacitor_SMD:C_0603_1608Metric -> Capacitor_SMD:C_0805_2012Metric
- renumbered C22 to C30, C23 to C31, C24 to C32, C25 to C34, C27 to C38, C28 to C39, C29 to C40, FB1 to FB5
Other:
- moved on the sheet: C30, C31, C32, C34, C36, C38, C39, C40, FB5

Commit message: big things are happening
Parts:
- added C32: 100n, Capacitor_SMD:C_0402_1005Metric, symbol Device:C
- FB5: footprint (none) -> Inductor_SMD:L_0805_2012Metric
- renumbered C32 to C31, C31 to C33, C36 to C35, C38 to C36, C39 to C37, C40 to C38
Connections:
- net +3V3: now also C31.1, C32.1
- net GND: now also C32.2
- net VDD3P3: no longer C31.1
Other:
- moved on the sheet: C30, C31, C33, FB5
