File: PCB/en_button.kicad_sch (KiCad schematic)
At the start: 5 parts, among them SW1 RST

Commit message: yeah just read the journal son
Parts:
- C15: footprint Capacitor_SMD:C_0603_1608Metric -> Capacitor_SMD:C_0805_2012Metric
Changed lines of the file:
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@@
 		(dnp no)
 		(fields_autoplaced yes)
-		(property "Reference" "#PWR012"
+		(property "Reference" "#PWR010"
 			(at 194.31 148.59 0)
 			(hide yes)
@@
 			(project "CTR-1"
 				(path "/59fb818d-89a2-4fec-918a-42976325079d/08fc498b-0362-4639-8258-6b1363fcdc91"
-					(reference "#PWR012")
+					(reference "#PWR010")
 					(unit 1)
 				)
@@
 			)
 		)
-		(property "Footprint" "Capacitor_SMD:C_0603_1608Metric"
+		(property "Footprint" "Capacitor_SMD:C_0805_2012Metric"
 			(at 180.0352 116.84 0)
 			(hide yes)
@@
 		(dnp no)
 		(fields_autoplaced yes)
-		(property "Reference" "#PWR011"
+		(property "Reference" "#PWR09"
 			(at 194.31 110.49 0)
 			(hide yes)
@@
 			(project "CTR-1"
 				(path "/59fb818d-89a2-4fec-918a-42976325079d/08fc498b-0362-4639-8258-6b1363fcdc91"
-					(reference "#PWR011")
+					(reference "#PWR09")
 					(unit 1)
 				)
@@
 		(dnp no)
 		(fields_autoplaced yes)
-		(property "Reference" "#PWR010"
+		(property "Reference" "#PWR08"
 			(at 186.69 124.46 0)
 			(hide yes)
@@
 			(project "CTR-1"
 				(path "/59fb818d-89a2-4fec-918a-42976325079d/08fc498b-0362-4639-8258-6b1363fcdc91"
-					(reference "#PWR010")
+					(reference "#PWR08")
 					(unit 1)
 				)
@@
 		(dnp no)
 		(fields_autoplaced yes)
-		(property "Reference" "#PWR09"
+		(property "Reference" "#PWR07"
 			(at 179.07 124.46 0)
 			(hide yes)
@@
 			(project "CTR-1"
 				(path "/59fb818d-89a2-4fec-918a-42976325079d/08fc498b-0362-4639-8258-6b1363fcdc91"
-					(reference "#PWR09")
-					(unit 1)
-				)
+					(reference "#PWR07")
+					(unit 1)
+				)

Commit message: big things are happening
Parts:
- R1: footprint (none) -> Resistor_SMD:R_0603_1608Metric; now in the parts list
Changed lines of the file:
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@@
 		(body_style 1)
 		(exclude_from_sim no)
-		(in_bom no)
-		(on_board no)
-		(in_pos_files no)
+		(in_bom yes)
+		(on_board yes)
+		(in_pos_files yes)
 		(dnp no)
 		(property "Reference" "R1"
@@
 			)
 		)
-		(property "Footprint" ""
+		(property "Footprint" "Resistor_SMD:R_0603_1608Metric"
 			(at 196.088 119.38 90)
 			(hide yes)
