File: PCB/gpio_cluster.kicad_sch (KiCad schematic)
At the start: 2 parts, among them J6 GPIO, J7 REF

Commit message: yeah just read the journal son
Parts:
- added C22: 100n, Capacitor_SMD:C_0603_1608Metric, symbol Device:C
- added C23: 10u, Capacitor_SMD:C_0805_2012Metric, symbol Device:C
- added FB1: 220@100MHz, symbol Device:FerriteBead
- J4: renamed from J7; footprint Connector_PinHeader_1.00mm:PinHeader_1x02_P1.00mm_Vertical -> Connector_PinHeader_2.54mm:PinHeader_1x02_P2.54mm_Vertical
- renumbered J6 to J3
Connections:
- net GND: now also C22.1, C23.1
- net cVDD: now also FB1.2; no longer J4.1 (Pin_1)
- new net: C22.2, C23.2, FB1.1, J4.1 (Pin_1)

Commit message: big things are happening
Parts:
- FB1: footprint (none) -> Inductor_SMD:L_0805_2012Metric
Changed lines of the file:
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@@
 			)
 		)
-		(property "Footprint" ""
+		(property "Footprint" "Inductor_SMD:L_0805_2012Metric"
 			(at 223.52 138.938 90)
 			(hide yes)
@@
 				)
 				(path "/59fb818d-89a2-4fec-918a-42976325079d/a6930468-3295-4954-a83d-ea3f44888009/8d5143ad-0f32-47f8-a7cc-18e0c8f4bcd8"
-					(reference "C42")
+					(reference "C40")
 					(unit 1)
 				)
@@
 				)
 				(path "/59fb818d-89a2-4fec-918a-42976325079d/a6930468-3295-4954-a83d-ea3f44888009/97701b60-d3a2-443e-91df-16d510ac3fdf"
-					(reference "C44")
+					(reference "C42")
 					(unit 1)
 				)
@@
 		(in_pos_files yes)
 		(dnp no)
-		(property "Reference" "#PWR025"
+		(property "Reference" "#PWR027"
 			(at 217.17 154.94 0)
 			(hide yes)
@@
 			(project "CTR-1"
 				(path "/59fb818d-89a2-4fec-918a-42976325079d/a6930468-3295-4954-a83d-ea3f44888009/2523cc3d-7b87-4688-8ee4-d8293bd6c074"
+					(reference "#PWR030")
+					(unit 1)
+				)
+				(path "/59fb818d-89a2-4fec-918a-42976325079d/a6930468-3295-4954-a83d-ea3f44888009/8d5143ad-0f32-47f8-a7cc-18e0c8f4bcd8"
+					(reference "#PWR039")
+					(unit 1)
+				)
+				(path "/59fb818d-89a2-4fec-918a-42976325079d/a6930468-3295-4954-a83d-ea3f44888009/9350a02e-2f10-4ecc-922a-85baace9d10a"
+					(reference "#PWR029")
+					(unit 1)
+				)
+				(path "/59fb818d-89a2-4fec-918a-42976325079d/a6930468-3295-4954-a83d-ea3f44888009/97701b60-d3a2-443e-91df-16d510ac3fdf"
+					(reference "#PWR042")
+					(unit 1)
+				)
+				(path "/59fb818d-89a2-4fec-918a-42976325079d/a6930468-3295-4954-a83d-ea3f44888009/c0cd88c9-43ea-4d15-a778-7f6969ee9636"
+					(reference "#PWR027")
+					(unit 1)
+				)
+				(path "/59fb818d-89a2-4fec-918a-42976325079d/a6930468-3295-4954-a83d-ea3f44888009/e5081cb5-7cd1-4fab-89e3-4b85fc1f336d"
 					(reference "#PWR028")
-					(unit 1)
-				)
-				(path "/59fb818d-89a2-4fec-918a-42976325079d/a6930468-3295-4954-a83d-ea3f44888009/8d5143ad-0f32-47f8-a7cc-18e0c8f4bcd8"
-					(reference "#PWR040")
-					(unit 1)
-				)
-				(path "/59fb818d-89a2-4fec-918a-42976325079d/a6930468-3295-4954-a83d-ea3f44888009/9350a02e-2f10-4ecc-922a-85baace9d10a"
-					(reference "#PWR027")
-					(unit 1)
-				)
-				(path "/59fb818d-89a2-4fec-918a-42976325079d/a6930468-3295-4954-a83d-ea3f44888009/97701b60-d3a2-443e-91df-16d510ac3fdf"
-					(reference "#PWR043")
-					(unit 1)
-				)
-				(path "/59fb818d-89a2-4fec-918a-42976325079d/a6930468-3295-4954-a83d-ea3f44888009/c0cd88c9-43ea-4d15-a778-7f6969ee9636"
-					(reference "#PWR025")
-					(unit 1)
-				)
-				(path "/59fb818d-89a2-4fec-918a-42976325079d/a6930468-3295-4954-a83d-ea3f44888009/e5081cb5-7cd1-4fab-89e3-4b85fc1f336d"
-					(reference "#PWR026")
 					(unit 1)
 				)
@@
 				)
 				(path "/59fb818d-89a2-4fec-918a-42976325079d/a6930468-3295-4954-a83d-ea3f44888009/8d5143ad-0f32-47f8-a7cc-18e0c8f4bcd8"
-					(reference "C41")
+					(reference "C39")
 					(unit 1)
 				)
@@
 				)
 				(path "/59fb818d-89a2-4fec-918a-42976325079d/a6930468-3295-4954-a83d-ea3f44888009/97701b60-d3a2-443e-91df-16d510ac3fdf"
-					(reference "C43")
-					(unit 1)
-				)
+					(reference "C41")
+					(unit 1)
+				)
