File: PCB/memory.kicad_sch (KiCad schematic)
At the start: 2 parts, among them U2 ESP-PSRAM64H

Commit message: yeah just read the journal son
Parts:
- added R11: 10k, symbol Device:R
- added U6: W25Q128JVE, Package_SON:WSON-8-1EP_8x6mm_P1.27mm_EP3.4x4.3mm, symbol Memory_Flash:W25Q128JVE
- renumbered U2 to U4
Connections:
- net GND: now also U6.4 (GND), U6.9 (EP)
- net SCLK: now also U6.6 (CLK)
- net SI/SIO: now also U6.5 (DI/IO_{0})
- net SIO2: now also U6.3 (~{WP}/IO_{2})
- net SIO3: now also U6.7 (~{HOLD}/~{RESET}/IO_{3})
- net SO/SIO: now also U6.2 (DO/IO_{1})
- net VCC: now also R11.2, U6.8 (VCC)
- net ~{CE} renamed ~{CE1}
- new net ~{CS0}: U6.1 (~{CS})

Commit message: big things are happening
Parts:
- removed R11, R4: 10k, symbol Device:R
- removed U4: ESP-PSRAM64H, Package_SO:SOIC-8_3.9x4.9mm_P1.27mm, symbol Memory_RAM:ESP-PSRAM32
- removed U6: W25Q128JVE, Package_SON:WSON-8-1EP_8x6mm_P1.27mm_EP3.4x4.3mm, symbol Memory_Flash:W25Q128JVE
- added R13, R14, R15, R16, R17: 0, Resistor_SMD:R_0402_1005Metric, symbol Device:R
Connections:
- net SCLK: now also R13.2
- net SI/SIO: now also R14.2
- net SIO2: now also R15.2
- net SIO3: now also R16.2
- net SO/SIO: now also R17.2
- new net FLASH/SCLK: R13.1
- new net FLASH/SI/SIO: R14.1
- new net FLASH/SIO2: R15.1
- new net FLASH/SIO3: R16.1
- new net FLASH/SO/SIO: R17.1
Other:
- added sheet FLASH (flash.kicad_sch)
- added sheet PSRAM (psram.kicad_sch)
