File: PCB/power_mgmt.kicad_sch (KiCad schematic)
At the start: 11 parts, among them U3 TPS259230, U5 AP2112K-3.3, U7 TVS1400DRV

Commit message: big things are happening
Parts:
- U7: renamed from U5; footprint PCM_SparkFun-Semiconductor-Standard:SOT23-5 -> Package_TO_SOT_SMD:SOT-23-5
- renumbered C45 to C43, C46 to C44, C33 to C45, C35 to C46, C37 to C47, R9 to R11, R10 to R12, U7 to U5, U3 to U6
Changed lines of the file:
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@@
 		(in_pos_files yes)
 		(dnp no)
-		(property "Reference" "#PWR046"
+		(property "Reference" "#PWR051"
 			(at 204.47 128.27 0)
 			(hide yes)
@@
 			(project "CTR-1"
 				(path "/59fb818d-89a2-4fec-918a-42976325079d/4ab54a93-ce3e-4d36-ab13-5a839d38f26c"
-					(reference "#PWR046")
+					(reference "#PWR051")
 					(unit 1)
 				)
@@
 		(in_pos_files yes)
 		(dnp no)
-		(property "Reference" "R10"
+		(property "Reference" "R12"
 			(at 196.85 135.89 0)
 			(show_name no)
@@
 			(project "CTR-1"
 				(path "/59fb818d-89a2-4fec-918a-42976325079d/4ab54a93-ce3e-4d36-ab13-5a839d38f26c"
-					(reference "R10")
+					(reference "R12")
 					(unit 1)
 				)
@@
 		(dnp no)
 		(fields_autoplaced yes)
-		(property "Reference" "#PWR049"
+		(property "Reference" "#PWR050"
 			(at 195.58 149.86 0)
 			(hide yes)
@@
 			(project "CTR-1"
 				(path "/59fb818d-89a2-4fec-918a-42976325079d/4ab54a93-ce3e-4d36-ab13-5a839d38f26c"
-					(reference "#PWR049")
+					(reference "#PWR050")
 					(unit 1)
 				)
@@
 		(in_pos_files yes)
 		(dnp no)
-		(property "Reference" "C37"
+		(property "Reference" "C47"
 			(at 233.68 132.08 0)
 			(show_name no)
@@
 			(project "CTR-1"
 				(path "/59fb818d-89a2-4fec-918a-42976325079d/4ab54a93-ce3e-4d36-ab13-5a839d38f26c"
-					(reference "C37")
+					(reference "C47")
 					(unit 1)
 				)
@@
 		(in_pos_files yes)
 		(dnp no)
-		(property "Reference" "#PWR015"
+		(property "Reference" "#PWR045"
 			(at 147.32 113.03 0)
 			(hide yes)
@@
 			(project "CTR-1"
 				(path "/59fb818d-89a2-4fec-918a-42976325079d/4ab54a93-ce3e-4d36-ab13-5a839d38f26c"
-					(reference "#PWR015")
+					(reference "#PWR045")
 					(unit 1)
 				)
@@
 		(in_pos_files yes)
 		(dnp no)
-		(property "Reference" "C33"
+		(property "Reference" "C45"
 			(at 207.01 130.81 0)
 			(show_name no)
@@
 			(project "CTR-1"
 				(path "/59fb818d-89a2-4fec-918a-42976325079d/4ab54a93-ce3e-4d36-ab13-5a839d38f26c"
-					(reference "C33")
+					(reference "C45")
 					(unit 1)
 				)
@@
 		(in_pos_files yes)
 		(dnp no)
-		(property "Reference" "C35"
+		(property "Reference" "C46"
 			(at 228.6 132.08 0)
 			(show_name no)
@@
 			(project "CTR-1"
 				(path "/59fb818d-89a2-4fec-918a-42976325079d/4ab54a93-ce3e-4d36-ab13-5a839d38f26c"
-					(reference "C35")
+					(reference "C46")
 					(unit 1)
 				)
@@
 		(dnp no)
 		(fields_autoplaced yes)
-		(property "Reference" "#PWR050"
+		(property "Reference" "#PWR048"
 			(at 189.23 149.86 0)
 			(hide yes)
@@
 			(project "CTR-1"
 				(path "/59fb818d-89a2-4fec-918a-42976325079d/4ab54a93-ce3e-4d36-ab13-5a839d38f26c"
-					(reference "#PWR050")
+					(reference "#PWR048")
 					(unit 1)
 				)
@@
 		(dnp no)
 		(fields_autoplaced yes)
-		(property "Reference" "U5"
+		(property "Reference" "U7"
 			(at 219.71 115.57 0)
 			(show_name no)
@@
 			)
 		)
-		(property "Footprint" "PCM_SparkFun-Semiconductor-Standard:SOT23-5"
+		(property "Footprint" "Package_TO_SOT_SMD:SOT-23-5"
 			(at 219.71 140.97 0)
 			(hide yes)
@@
 			(project "CTR-1"
 				(path "/59fb818d-89a2-4fec-918a-42976325079d/4ab54a93-ce3e-4d36-ab13-5a839d38f26c"
-					(reference "U5")
+					(reference "U7")
 					(unit 1)
 				)
@@
 		(in_pos_files yes)
 		(dnp no)
-		(property "Reference" "#PWR031"
+		(property "Reference" "#PWR049"
 			(at 195.58 128.27 0)
 			(hide yes)
@@
 			(project "CTR-1"
 				(path "/59fb818d-89a2-4fec-918a-42976325079d/4ab54a93-ce3e-4d36-ab13-5a839d38f26c"
-					(reference "#PWR031")
+					(reference "#PWR049")
 					(unit 1)
 				)
@@
 		(dnp no)
 		(fields_autoplaced yes)
-		(property "Reference" "#PWR037"
+		(property "Reference" "#PWR053"
 			(at 236.22 128.27 0)
 			(hide yes)
@@
 			(project "CTR-1"
 				(path "/59fb818d-89a2-4fec-918a-42976325079d/4ab54a93-ce3e-4d36-ab13-5a839d38f26c"
-					(reference "#PWR037")
+					(reference "#PWR053")
 					(unit 1)
 				)
@@
 		(dnp no)
 		(fields_autoplaced yes)
-		(property "Reference" "#PWR034"
+		(property "Reference" "#PWR052"
 			(at 219.71 149.86 0)
 			(hide yes)
@@
 			(project "CTR-1"
 				(path "/59fb818d-89a2-4fec-918a-42976325079d/4ab54a93-ce3e-4d36-ab13-5a839d38f26c"
-					(reference "#PWR034")
+					(reference "#PWR052")
 					(unit 1)
 				)
@@
 		(in_pos_files yes)
 		(dnp no)
-		(property "Reference" "C46"
+		(property "Reference" "C44"
 			(at 189.23 137.16 0)
 			(show_name no)
@@
 			(project "CTR-1"
 				(path "/59fb818d-89a2-4fec-918a-42976325079d/4ab54a93-ce3e-4d36-ab13-5a839d38f26c"
-					(reference "C46")
+					(reference "C44")
 					(unit 1)
 				)
@@
 		(in_pos_files yes)
 		(dnp no)
-		(property "Reference" "C45"
+		(property "Reference" "C43"
 			(at 153.67 129.54 0)
 			(show_name no)
@@
 			(project "CTR-1"
 				(path "/59fb818d-89a2-4fec-918a-42976325079d/4ab54a93-ce3e-4d36-ab13-5a839d38f26c"
-					(reference "C45")
+					(reference "C43")
 					(unit 1)
 				)
@@
 		(in_pos_files yes)
 		(dnp no)
-		(property "Reference" "U3"
+		(property "Reference" "U6"
 			(at 170.18 124.46 0)
 			(show_name no)
@@
 			(project "CTR-1"
 				(path "/59fb818d-89a2-4fec-918a-42976325079d/4ab54a93-ce3e-4d36-ab13-5a839d38f26c"
-					(reference "U3")
+					(reference "U6")
 					(unit 1)
 				)
@@
 		(in_pos_files yes)
 		(dnp no)
-		(property "Reference" "U7"
+		(property "Reference" "U5"
 			(at 147.32 137.16 0)
 			(show_name no)
@@
 			(project "CTR-1"
 				(path "/59fb818d-89a2-4fec-918a-42976325079d/4ab54a93-ce3e-4d36-ab13-5a839d38f26c"
-					(reference "U7")
+					(reference "U5")
 					(unit 1)
 				)
@@
 		(dnp no)
 		(fields_autoplaced yes)
-		(property "Reference" "#PWR047"
+		(property "Reference" "#PWR046"
 			(at 147.32 149.86 0)
 			(hide yes)
@@
 			(project "CTR-1"
 				(path "/59fb818d-89a2-4fec-918a-42976325079d/4ab54a93-ce3e-4d36-ab13-5a839d38f26c"
-					(reference "#PWR047")
+					(reference "#PWR046")
 					(unit 1)
 				)
@@
 		(dnp no)
 		(fields_autoplaced yes)
-		(property "Reference" "#PWR048"
+		(property "Reference" "#PWR047"
 			(at 177.8 149.86 0)
 			(hide yes)
@@
 			(project "CTR-1"
 				(path "/59fb818d-89a2-4fec-918a-42976325079d/4ab54a93-ce3e-4d36-ab13-5a839d38f26c"
-					(reference "#PWR048")
+					(reference "#PWR047")
 					(unit 1)
 				)
@@
 		(in_pos_files yes)
 		(dnp no)
-		(property "Reference" "R9"
+		(property "Reference" "R11"
 			(at 161.29 125.73 0)
 			(show_name no)
@@
 			(project "CTR-1"
 				(path "/59fb818d-89a2-4fec-918a-42976325079d/4ab54a93-ce3e-4d36-ab13-5a839d38f26c"
-					(reference "R9")
-					(unit 1)
-				)
+					(reference "R11")
+					(unit 1)
+				)
