File: PCB/usb_c.kicad_sch (KiCad schematic)
At the start: 3 parts, among them J3 USB_C_Receptacle_USB2.0_16P

Commit message: yeah just read the journal son
Parts:
- added U2: USBLC6-2P6, Package_TO_SOT_SMD:SOT-666, symbol Power_Protection:USBLC6-2P6
- J2: renamed from J3; footprint (none) -> Connector_USB:USB_C_Receptacle_GCT_USB4105-xx-A_16P_TopMnt_Horizontal
- R2, R3: value R -> 5.1k; footprint (none) -> Resistor_SMD:R_0805_2012Metric
Connections:
- net D+: now also U2.4 (I/O2); no longer J2.A6 (D+), J2.B6 (D+)
- net D-: now also U2.6 (I/O1); no longer J2.A7 (D-), J2.B7 (D-)
- net GND: now also U2.2 (GND)
- new net: J2.A7 (D-), J2.B7 (D-), U2.1 (I/O1)
- new net: J2.A6 (D+), J2.B6 (D+), U2.3 (I/O2)
- new net VREG: U2.5 (VBUS)
