File: PCB/xtal_32k_rtc.kicad_sch (KiCad schematic)
At the start: 3 parts, among them Y2 32kHz

Commit message: big things are happening
Parts:
- removed C13, C14: MATCH, Capacitor_SMD:C_0603_1608Metric, symbol Device:C
- Y2: value 32kHz -> 32.768kHz; footprint (none) -> Crystal:Crystal_SMD_3225-4Pin_3.2x2.5mm
