File: PCB/CTR-1.kicad_pcb (KiCad board)
At the start: 4 copper layers, 89 parts, among them J1 u.FL, J10 REF, J11 GPIO, J12 REF, J13 REF, J14 JTAG, J15 GPIO, J16 REF, J17 UART, J2 USB_C_Receptacle_USB2.0_16P, J3 GPIO, J4 REF, J5 GPIO, J6 REF, J7 GPIO, J8 REF, J9 GPIO, SW1 RST, SW2 BOOT, SW3 BOOT, SW4 BOOT, U1 ESP32-S3, U2 USBLC6-2P6, U3 ESP-PSRAM64H, U4 W25Q128JVS, U5 TVS1400DRV, U6 TPS259230, U7 AP2112K-3.3, Y1 40MHz, Y2 32.768kHz

Commit message: sync
Parts:
- moved C42 230.2 mm to (97.0, 114.2), turned to -90 degrees
- moved FB7 228.5 mm to (97.0, 118.7), turned to -90 degrees
- moved J11 227.6 mm to (74.9, 147.9), turned to 90 degrees
- moved J12 227.2 mm to (68.8, 147.9), turned to 90 degrees
- moved C41 227.1 mm to (97.0, 123.0), turned to -90 degrees
- moved J16 222.1 mm to (97.0, 108.6), turned to 180 degrees
- moved C40 218.4 mm to (63.2, 147.9), turned to 180 degrees
- moved J15 215.9 mm to (97.0, 102.5), turned to 180 degrees
- moved FB6 211.8 mm to (58.7, 147.9), turned to 180 degrees
- moved C39 205.7 mm to (54.4, 147.9), turned to 180 degrees
- moved C22 198.6 mm to (89.7, 41.0)
- moved FB1 198.6 mm to (85.4, 41.0)
- moved C23 198.6 mm to (80.9, 41.0)
- moved J4 196.6 mm to (75.3, 41.0), turned to -90 degrees
- moved J3 189.2 mm to (69.2, 41.0), turned to -90 degrees
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Routing:
- net /ESP32-S3 MCU/MTCK: track 4.81 -> 22.2 mm
- net /ESP32-S3 MCU/MTMS: track 4.81 -> 21.8 mm
- net /ESP32-S3 MCU/MTDO: track 4.87 -> 21.0 mm
- net /ESP32-S3 MCU/MTDI: track 4.90 -> 20.9 mm
- net /ESP32-S3 MCU/XTAL_32K_P: track 6.26 -> 0.00 mm
- net /ESP32-S3 MCU/XTAL_32K_N: track 5.90 -> 0.00 mm
- net VDD3P3_RTC: track 21.2 -> 22.7 mm
- net /GPIO45: track 0.00 -> 1.19 mm, vias 0 -> 1
- net /ESP32-S3 MCU/GPIO21: track 0.00 -> 1.14 mm, vias 0 -> 1
- net /ESP32-S3 MCU/GPIO36: track 0.00 -> 1.09 mm, vias 0 -> 1
- net /ESP32-S3 MCU/GPIO34: track 0.00 -> 1.08 mm, vias 0 -> 1
- net /ESP32-S3 MCU/GPIO17: track 0.00 -> 1.04 mm, vias 0 -> 1
- net /ESP32-S3 MCU/GPIO11: track 0.00 -> 1.04 mm, vias 0 -> 1
- net /ESP32-S3 MCU/GPIO13: track 0.00 -> 1.04 mm, vias 0 -> 1
- net /ESP32-S3 MCU/GPIO1: track 0.00 -> 1.01 mm, vias 0 -> 1
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